Commit message: fixed bugs from project 2

File: my_robot/urdf/my_robot.xacro (robot description, xacro)
@@ -12,12 +12,4 @@
     <inertia ixx="${2*m*r*r/5}" ixy = "0" ixz = "0" iyy="${2*m*r*r/5}" iyz = "0" izz="${2*m*r*r/5}" />
   </xacro:macro>
-  <xacro:property name="wheel_mass" value="0.5" />
-  <xacro:property name="wheel_radius" value="0.12" />
-  <xacro:property name="wheel_length" value="0.05" />
-  <xacro:property name="caster_radius" value="0.03" />
-  <xacro:property name="base_x_len" value="0.2" />
-  <xacro:property name="base_y_len" value="0.3" />
-  <xacro:property name="base_z_len" value="0.14" />
-  <xacro:property name="base_chassis_mass" value="10" />
   <link name="robot_footprint"></link>
   <xacro:include filename="$(find my_robot)/urdf/my_robot.gazebo" />
@@ -30,12 +22,13 @@
     <pose>0 0 0.12 0 0 0</pose>
     <inertial>
-      <mass value="${base_chassis_mass}"/>
-      <origin xyz="0 0 0" rpy=" 0 0 0"/>
-      <cuboid_inertia m="${base_chassis_mass}" x= "${base_x_len}" y= "${base_y_len}" z="${base_z_len}"/>
+      <mass value="10"/>
+      <origin xyz="0 0 0" rpy=" 0 0 0"/>
+      <cuboid_inertia m="10" x= "0.2" y= "0.3" z="0.14"/>
+      <inertia ixx="0.09133" ixy = "0" ixz = "0" iyy="0.04967" iyz = "0" izz="0.0685" />
     </inertial>
     <collision name='collision'>
       <origin xyz="0 0 0" rpy=" 0 0 0"/>
       <geometry>
-        <box size="${base_x_len} ${base_y_len} ${base_z_len}"/>
+        <box size="0.2 0.3 0.14"/>
       </geometry>
     </collision>
@@ -43,5 +36,5 @@
       <origin xyz="0 0 0" rpy=" 0 0 0"/>
       <geometry>
-        <box size="${base_x_len} ${base_y_len} ${base_z_len}"/>
+        <box size="0.2 0.3 0.14"/>
       </geometry>
     </visual>
@@ -51,10 +44,10 @@
       <mass value="0.01"/>
       <origin xyz="0 0 0" rpy=" 0 0 0"/>
-      <cuboid_inertia m="0.01" x= "${base_x_len}" y= "0.1" z="0.1"/>
+      <inertia ixx="0.000016667" ixy = "0" ixz = "0" iyy="0.00004167" iyz = "0" izz="0.00004167" />
     </inertial>
     <collision name='collision'>
       <origin xyz="0 0 0" rpy=" 0 0 0"/>
       <geometry>
-        <box size="${base_x_len} 0.1 0.1"/>
+        <box size="0.2 0.1 0.1"/>
       </geometry>
     </collision>
@@ -62,5 +55,5 @@
       <origin xyz="0 0 0" rpy=" 0 0 0"/>
       <geometry>
-        <box size="${base_x_len} 0.1 0.1"/>
+        <box size="0.2 0.1 0.1"/>
       </geometry>
     </visual>
@@ -73,12 +66,13 @@
 <link name='sup_chassis'>
   <inertial>
-    <mass value="${base_chassis_mass/3}"/>
-    <origin xyz="0 0 0" rpy=" 0 0 0"/>
-    <cuboid_inertia m="${base_chassis_mass/3}" x= "${base_x_len*1.5}" y= "${base_y_len}" z="0.05"/>
-  </inertial>
-  <collision name='collision'>
-    <origin xyz="0 0 0" rpy=" 0 0 0"/>
-    <geometry>
-      <box size="${base_x_len*1.5} ${base_y_len} 0.05"/>
+    <mass value="3"/>
+    <origin xyz="0 0 0" rpy=" 0 0 0"/>
+    <cuboid_inertia m="3" x= "0.3" y= "0.3" z="0.05"/>
+    <inertia ixx="0.023125" ixy = "0" ixz = "0" iyy="0.023125" iyz = "0" izz="0.045" />
+  </inertial>
+  <collision name='collision'>
+    <origin xyz="0 0 0" rpy=" 0 0 0"/>
+    <geometry>
+      <box size="0.3 0.3 0.05"/>
     </geometry>
   </collision>
@@ -86,22 +80,22 @@
     <origin xyz="0 0 0" rpy=" 0 0 0"/>
     <geometry>
-      <box size="${base_x_len*1.5} ${base_y_len} 0.05"/>
+      <box size="0.3 0.3 0.05"/>
     </geometry>
   </visual>
   <collision name='caster_collision'>
-    <origin xyz="${-base_x_len*3/4 + caster_radius} 0 -0.025" rpy=" 0 0 0"/>
-    <geometry>
-      <sphere radius="${caster_radius-0.001}"/>
+    <origin xyz="-0.12 0 -0.025" rpy=" 0 0 0"/>
+    <geometry>
+      <sphere radius="0.029"/>
     </geometry>
   </collision>
   <visual name='caster_visual'>
-    <origin xyz="${-base_x_len*3/4 + caster_radius} 0 -0.025" rpy=" 0 0 0"/>
-    <geometry>
-      <sphere radius="${caster_radius}"/>
+    <origin xyz="-0.12 0 -0.025" rpy=" 0 0 0"/>
+    <geometry>
+      <sphere radius="0.03"/>
     </geometry>
   </visual>
 </link>
 <joint type="fixed" name="sup_chassis_joint">
-  <origin xyz="${-base_x_len*5/4} 0 -0.045" rpy="0 0 0"/>
+  <origin xyz="-0.25 0 -0.045" rpy="0 0 0"/>
   <child link="sup_chassis"/>
   <parent link="base_chassis"/>
@@ -112,10 +106,10 @@
     <mass value="0.1"/>
     <origin xyz="0 0 0" rpy=" 0 0 0"/>
-    <cuboid_inertia m="0.1" x= "0.01" y= "${base_y_len}" z="0.05"/>
-  </inertial>
-  <collision name='collision'>
-    <origin xyz="0 0 0" rpy=" 0 0 0"/>
-    <geometry>
-      <box size="0.01 ${base_y_len} 0.05"/>
+    <inertia ixx="0.0007708" ixy = "0" ixz = "0" iyy="0.000021667" iyz = "0" izz="0.0007508" />
+  </inertial>
+  <collision name='collision'>
+    <origin xyz="0 0 0" rpy=" 0 0 0"/>
+    <geometry>
+      <box size="0.01 0.3 0.05"/>
     </geometry>
   </collision>
@@ -123,10 +117,10 @@
     <origin xyz="0 0 0" rpy=" 0 0 0"/>
     <geometry>
-      <box size="0.01 ${base_y_len} 0.05"/>
+      <box size="0.01 0.3 0.05"/>
     </geometry>
   </visual>
 </link>
 <joint type="fixed" name="back_sup_chassis_joint">
-  <origin xyz="${-base_x_len*3/4 - 0.005} 0 0" rpy="0 0 0"/>
+  <origin xyz="-0.155 0 0" rpy="0 0 0"/>
   <child link="back_sup_chassis"/>
   <parent link="sup_chassis"/>
@@ -135,12 +129,12 @@
 <link name='left_wheel'>
   <inertial>
-    <mass value="${wheel_mass}"/>
-    <origin xyz="0.0 0 0" rpy=" 0 1.5707 1.5707"/>
-    <cylinder_inertia m="${wheel_mass}" r= "${wheel_radius}" l= "${wheel_length}"/>
-  </inertial>
-  <collision name='collision'>
-    <origin xyz="0.0 0 0" rpy=" 0 1.5707 1.5707"/>
-    <geometry>
-      <cylinder radius="${wheel_radius}" length="${wheel_length}" />
+    <mass value="0.5"/>
+    <origin xyz="0.0 0 0" rpy=" 0 1.5707 1.5707"/>
+    <inertia ixx="0.001904" ixy = "0" ixz = "0" iyy="0.001904" iyz = "0" izz="0.0036" />
+  </inertial>
+  <collision name='collision'>
+    <origin xyz="0.0 0 0" rpy=" 0 1.5707 1.5707"/>
+    <geometry>
+      <cylinder radius="0.12" length="0.05" />
     </geometry>
   </collision>
@@ -148,5 +142,5 @@
     <origin xyz="0.0 0 0" rpy=" 0 1.5707 1.5707"/>
     <geometry>
-      <cylinder radius="${wheel_radius}" length="${wheel_length}" />
+      <cylinder radius="0.12" length="0.05" />
     </geometry>
   </visual>
@@ -154,12 +148,12 @@
 <link name='right_wheel'>
   <inertial>
-    <mass value="${wheel_mass}"/>
-    <origin xyz="0.0 0 0" rpy=" 0 1.5707 1.5707"/>
-    <cylinder_inertia m="${wheel_mass}" r= "${wheel_radius}" l= "${wheel_length}"/>
-  </inertial>
-  <collision name='collision'>
-    <origin xyz="0.0 0 0" rpy=" 0 1.5707 1.5707"/>
-    <geometry>
-      <cylinder radius="${wheel_radius}" length="${wheel_length}" />
+    <mass value="0.5"/>
+    <origin xyz="0.0 0 0" rpy=" 0 1.5707 1.5707"/>
+    <inertia ixx="0.001904" ixy = "0" ixz = "0" iyy="0.001904" iyz = "0" izz="0.0036" />
+  </inertial>
+  <collision name='collision'>
+    <origin xyz="0.0 0 0" rpy=" 0 1.5707 1.5707"/>
+    <geometry>
+      <cylinder radius="0.12" length="0.05" />
     </geometry>
   </collision>
@@ -167,10 +161,10 @@
     <origin xyz="0.0 0 0" rpy=" 0 1.5707 1.5707"/>
     <geometry>
-      <cylinder radius="${wheel_radius}" length="${wheel_length}" />
+      <cylinder radius="0.12" length="0.05" />
     </geometry>
   </visual>
 </link>
 <joint type="continuous" name="left_wheel_hinge">
-  <origin xyz="0 ${(base_y_len + wheel_length)/2 +0.01} 0.02" rpy="0 0 0"/>
+  <origin xyz="0 0.185 0.02" rpy="0 0 0"/>
   <child link="left_wheel"/>
   <parent link="base_chassis"/>
@@ -180,5 +174,5 @@
 </joint>
 <joint type="continuous" name="right_wheel_hinge">
-  <origin xyz="0 ${-1*(base_y_len + wheel_length)/2 -0.01} 0.02" rpy="0 0 0"/>
+  <origin xyz="0 -0.185 0.02" rpy="0 0 0"/>
   <child link="right_wheel"/>
   <parent link="base_chassis"/>
@@ -208,5 +202,5 @@
 </link>
 <joint type="fixed" name="camera_joint">
-  <origin xyz="${base_x_len/2 +0.025} 0 0" rpy="0 0 0"/>
+  <origin xyz="0.125 0 0" rpy="0 0 0"/>
   <child link="camera"/>
   <parent link="base_chassis"/>
